Commit message: Added mcm07_husky customization and integrated OAK-D

File: catkin_ws/src/husky_oakd_stereo_nav/urdf/oak-d.urdf.xacro (robot description, xacro)
@@ -19,390 +19,258 @@
   <!-- Xacro property for IMU -->
   <xacro:property name="imu_update_rate" value="100" /> <!-- IMU update rate in Hz (reasonable default) -->
-  <!-- Stand base plate (30cm above top_plate_link, 20cm wide, 40cm deep, 1cm thick) -->
-  <link name="camera_stand_base">
-    <visual>
-      <origin xyz="0 0 0" rpy="0 0 0" />
-      <geometry>
-        <box size="0.20 0.40 0.01" /> <!-- 20cm wide, 40cm deep, 1cm thick -->
-      </geometry>
-      <material name="silver">
-        <color rgba="0.7 0.7 0.7 1.0" />
-      </material>
-    </visual>
-    <collision>
-      <origin xyz="0 0 0" rpy="0 0 0" />
-      <geometry>
-        <box size="0.20 0.40 0.01" />
-      </geometry>
-    </collision>
-    <inertial>
-      <mass value="0.3" />
-      <inertia ixx="0.004" ixy="0" ixz="0" iyy="0.013" iyz="0" izz="0.004" />
-    </inertial>
-  </link>
-  <!-- Four support props (30cm tall, 2cm diameter) -->
-  <link name="stand_prop_1">
-    <visual>
-      <origin xyz="0 0 0" rpy="0 0 0" />
-      <geometry>
-        <cylinder radius="0.01" length="0.30" />
-      </geometry>
-      <material name="silver" />
-    </visual>
-    <collision>
-      <origin xyz="0 0 0" rpy="0 0 0" />
-      <geometry>
-        <cylinder radius="0.01" length="0.30" />
-      </geometry>
-    </collision>
-    <inertial>
-      <mass value="0.1" />
-      <inertia ixx="0.001" ixy="0" ixz="0" iyy="0.001" iyz="0" izz="0.0001" />
-    </inertial>
-  </link>
-  <link name="stand_prop_2">
-    <visual>
-      <origin xyz="0 0 0" rpy="0 0 0" />
-      <geometry>
-        <cylinder radius="0.01" length="0.30" />
-      </geometry>
-      <material name="silver" />
-    </visual>
-    <collision>
-      <origin xyz="0 0 0" rpy="0 0 0" />
-      <geometry>
-        <cylinder radius="0.01" length="0.30" />
-      </geometry>
-    </collision>
-    <inertial>
-      <mass value="0.1" />
-      <inertia ixx="0.001" ixy="0" ixz="0" iyy="0.001" iyz="0" izz="0.0001" />
-    </inertial>
-  </link>
-  <link name="stand_prop_3">
-    <visual>
-      <origin xyz="0 0 0" rpy="0 0 0" />
-      <geometry>
-        <cylinder radius="0.01" length="0.30" />
-      </geometry>
-      <material name="silver" />
-    </visual>
-    <collision>
-      <origin xyz="0 0 0" rpy="0 0 0" />
-      <geometry>
-        <cylinder radius="0.01" length="0.30" />
-      </geometry>
-    </collision>
-    <inertial>
-      <mass value="0.1" />
-      <inertia ixx="0.001" ixy="0" ixz="0" iyy="0.001" iyz="0" izz="0.0001" />
-    </inertial>
-  </link>
-  <link name="stand_prop_4">
-    <visual>
-      <origin xyz="0 0 0" rpy="0 0 0" />
-      <geometry>
-        <cylinder radius="0.01" length="0.30" />
-      </geometry>
-      <material name="silver" />
-    </visual>
-    <collision>
-      <origin xyz="0 0 0" rpy="0 0 0" />
-      <geometry>
-        <cylinder radius="0.01" length="0.30" />
-      </geometry>
-    </collision>
-    <inertial>
-      <mass value="0.1" />
-      <inertia ixx="0.001" ixy="0" ixz="0" iyy="0.001" iyz="0" izz="0.0001" />
-    </inertial>
-  </link>
-  <!-- Joints connecting stand to top_plate_link -->
-  <joint name="stand_base_joint" type="fixed">
-    <parent link="top_plate_link" />
-    <child link="camera_stand_base" />
-    <origin xyz="0 0 0.305" rpy="0 0 0" /> <!-- 30.5cm up to center of 1cm thick plate -->
-  </joint>
-  <joint name="prop_1_joint" type="fixed">
-    <parent link="top_plate_link" />
-    <child link="stand_prop_1" />
-    <origin xyz="0.08 0.18 0.15" rpy="0 0 0" /> <!-- Front-left corner -->
-  </joint>
-  <joint name="prop_2_joint" type="fixed">
-    <parent link="top_plate_link" />
-    <child link="stand_prop_2" />
-    <origin xyz="0.08 -0.18 0.15" rpy="0 0 0" /> <!-- Front-right corner -->
-  </joint>
-  <joint name="prop_3_joint" type="fixed">
-    <parent link="top_plate_link" />
-    <child link="stand_prop_3" />
-    <origin xyz="-0.08 0.18 0.15" rpy="0 0 0" /> <!-- Rear-left corner -->
-  </joint>
-  <joint name="prop_4_joint" type="fixed">
-    <parent link="top_plate_link" />
-    <child link="stand_prop_4" />
-    <origin xyz="-0.08 -0.18 0.15" rpy="0 0 0" /> <!-- Rear-right corner -->
-  </joint>
-  <!-- Camera links -->
-  <!-- Oak-D Camera Integration -->
-  <link name="oak-d-base-frame"/>
-  <!-- Joint connecting Oak-D base to stand -->
-  <joint name="oak_d_base_joint" type="fixed">
-    <parent link="camera_stand_base" />
-    <child link="oak-d-base-frame" />
-    <origin xyz="0.10 0 0.0495" rpy="0 0 0" /> <!-- Front edge of stand, centered on 1cm thick plate -->
-    <!-- Dimensions: 110x54.5x33 mm  -->
-  </joint>
-  <!-- Oak-D base_link of the sensor -->
-  <link name="oak-d_frame"/>
-  <joint name="oak_center_joint" type="fixed">
-    <parent link="oak-d-base-frame"/>
-    <child link="oak-d_frame"/>
-    <origin rpy="0.0 0.0 0.0" xyz="0.0 0.0 0.0"/>
-  </joint>
-  <link name="oak_model_origin">
-    <visual>
+  <xacro:macro name="OAK-D" params="*origin parent:=oak-d-base-frame">
+    <!-- Camera links -->
+    <!-- Oak-D base_link of the sensor -->
+    <link name="oak-d_frame"/>
+    <joint name="oak_center_joint" type="fixed">
+      <parent link="${parent}"/>
+      <child link="oak-d_frame"/>
+      <origin rpy="0.0 0.0 0.0" xyz="0.0 0.0 0.0"/>
+    </joint>
+    <link name="oak_model_origin">
+      <visual>
+        <origin rpy="0 0 0" xyz="0 0 0"/>
+        <geometry>
+          <mesh filename="package://depthai_descriptions/urdf/models/OAK-D.stl"/>
+        </geometry>
+        <material name="mat">
+          <color rgba="0.8 0.8 0.8 0.8"/>
+        </material>
+      </visual>
+    </link>
+    <joint name="oak_model_origin_joint" type="fixed">
+      <parent link="oak-d_frame"/>
+      <child link="oak_model_origin"/>
+      <origin rpy="1.5708 0 1.5708" xyz="0 0 0"/>
+    </joint>
+    <!-- IMU -->
+    <link name="oak_imu_frame"/>
+    <joint name="oak_imu_joint" type="fixed">
+      <parent link="oak-d_frame"/>
+      <child link="oak_imu_frame"/>
+      <origin xyz="0.0 -0.015 -0.013662" rpy="0.0 1.5707963267948966 0.0"/>
+    </joint>
+    <xacro:if value="${imu_enabled}">
+      <!-- Gazebo plugin for IMU -->
+      <gazebo reference="oak_imu_frame">
+        <gravity>true</gravity>
+        <sensor name="imu_sensor" type="imu">
+          <always_on>true</always_on>
+          <update_rate>${imu_update_rate}</update_rate>
+          <visualize>true</visualize>
+          <topic>__default_topic__</topic>
+          <plugin filename="libgazebo_ros_imu_sensor.so" name="imu_plugin">
+            <topicName>/oak_d/imu</topicName>
+            <bodyName>oak_imu_frame</bodyName>
+            <updateRateHZ>${imu_update_rate}</updateRateHZ>
+            <gaussianNoise>0.0</gaussianNoise>
+            <xyzOffset>0 0 0</xyzOffset>
+            <rpyOffset>0 0 0</rpyOffset>
+            <frameName>oak_imu_frame</frameName>
+            <initialOrientationAsReference>false</initialOrientationAsReference>
+          </plugin>
+          <pose>0 0 0 0 0 0</pose>
+        </sensor>
+      </gazebo>
+    </xacro:if>
+    <!-- RGB Camera -->
+    <link name="oak_rgb_camera_frame"/>
+    <joint name="oak_rgb_camera_joint" type="fixed">
+      <parent link="oak-d_frame"/>
+      <child link="oak_rgb_camera_frame"/>
       <origin rpy="0 0 0" xyz="0 0 0"/>
-      <geometry>
-        <mesh filename="package://depthai_descriptions/urdf/models/OAK-D.stl"/>
-      </geometry>
-      <material name="mat">
-        <color rgba="0.8 0.8 0.8 0.8"/>
-      </material>
-    </visual>
-  </link>
-  <joint name="oak_model_origin_joint" type="fixed">
-    <parent link="oak-d_frame"/>
-    <child link="oak_model_origin"/>
-    <origin rpy="1.5708 0 1.5708" xyz="0 0 0"/>
-  </joint>
-  <!-- IMU -->
-  <link name="oak_imu_frame"/>
-  <joint name="oak_imu_joint" type="fixed">
-    <parent link="oak-d_frame"/>
-    <child link="oak_imu_frame"/>
-    <origin rpy="0.0 1.5707963267948966 0.0" xyz="0.0 -0.015 -0.013662"/>
-  </joint>
-  <xacro:if value="${imu_enabled}">
-    <!-- Gazebo plugin for IMU -->
-    <gazebo reference="oak_imu_frame">
-      <gravity>true</gravity>
-      <sensor name="imu_sensor" type="imu">
-        <always_on>true</always_on>
-        <update_rate>${imu_update_rate}</update_rate>
-        <visualize>true</visualize>
-        <topic>__default_topic__</topic>
-        <plugin filename="libgazebo_ros_imu_sensor.so" name="imu_plugin">
-          <topicName>/oak_d/imu</topicName>
-          <bodyName>oak_imu_frame</bodyName>
-          <updateRateHZ>${imu_update_rate}</updateRateHZ>
-          <gaussianNoise>0.0</gaussianNoise>
-          <xyzOffset>0 0 0</xyzOffset>
-          <rpyOffset>0 0 0</rpyOffset>
-          <frameName>oak_imu_frame</frameName>
-          <initialOrientationAsReference>false</initialOrientationAsReference>
-        </plugin>
-        <pose>0 0 0 0 0 0</pose>
-      </sensor>
-    </gazebo>
-  </xacro:if>
-  <!-- RGB Camera -->
-  <link name="oak_rgb_camera_frame"/>
-  <joint name="oak_rgb_camera_joint" type="fixed">
-    <parent link="oak-d_frame"/>
-    <child link="oak_rgb_camera_frame"/>
-    <origin rpy="0 0 0" xyz="0 0 0"/>
-  </joint>
-  <link name="oak_rgb_camera_optical_frame"/>
-  <joint name="oak_rgb_camera_optical_joint" type="fixed">
-    <origin rpy="-1.5707963267948966 0.0 -1.5707963267948966" xyz="0 0 0"/>
-    <parent link="oak_rgb_camera_frame"/>
-    <child link="oak_rgb_camera_optical_frame"/>
-  </joint>
-  <!-- Left Camera -->
-  <link name="oak_left_camera_frame"/>
-  <joint name="oak_left_camera_joint" type="fixed">
-    <parent link="oak-d_frame"/>
-    <child link="oak_left_camera_frame"/>
-    <origin rpy="0 0 0" xyz="0 0.0375 0"/>
-  </joint>
-  <link name="oak_left_camera_optical_frame"/>
-  <joint name="oak_left_camera_optical_joint" type="fixed">
-    <origin rpy="-1.5707963267948966 0.0 -1.5707963267948966" xyz="0 0 0"/>
-    <parent link="oak_left_camera_frame"/>
-    <child link="oak_left_camera_optical_frame"/>
-  </joint>
-  <!-- Right Camera -->
-  <link name="oak_right_camera_frame"/>
-  <joint name="oak_right_camera_joint" type="fixed">
-    <parent link="oak-d_frame"/>
-    <child link="oak_right_camera_frame"/>
-    <origin rpy="0 0 0" xyz="0 -0.0375 0"/>
-  </joint>
-  <link name="oak_right_camera_optical_frame"/>
-  <joint name="oak_right_camera_optical_joint" type="fixed">
-    <origin rpy="-1.5707963267948966 0.0 -1.5707963267948966" xyz="0 0 0"/>
-    <parent link="oak_right_camera_frame"/>
-    <child link="oak_right_camera_optical_frame"/>
-  </joint>
-  <xacro:if value="${rgb_camera_enabled}">
-    <!-- Gazebo plugin for RGB Camera -->
-    <gazebo reference="oak_rgb_camera_frame">
-      <sensor type="camera" name="oak_rgb_sensor">
-        <update_rate>${rgb_update_rate}</update_rate>
-        <camera>
-          <horizontal_fov>1.2042771838760875</horizontal_fov> <!-- 69° HFOV in radians -->
-          <vertical_fov>0.9599310885968813</vertical_fov><!-- 55° VFOV in radians -->
-          <image>
-            <width>${rgb_width}</width>
-            <height>${rgb_height}</height>
-            <format>R8G8B8</format> <!-- Color camera -->
-          </image>
-          <clip>
-            <near>0.08</near> <!-- Min focus 8cm -->
-            <far>100.0</far> <!-- Arbitrary max range -->
-          </clip>
-        </camera>
-        <plugin name="oak_rgb_camera_controller" filename="libgazebo_ros_camera.so">
-          <alwaysOn>true</alwaysOn>
-          <updateRate>${rgb_update_rate}</updateRate>
-          <cameraName>oak_rgb</cameraName>
-          <frameName>oak_rgb_camera_optical_frame</frameName>
-          <imageTopicName>image_raw</imageTopicName>
-          <cameraInfoTopicName>camera_info</cameraInfoTopicName>
-          <distortionK1>0.0</distortionK1>
-          <distortionK2>0.0</distortionK2>
-          <distortionK3>0.0</distortionK3>
-          <distortionT1>0.0</distortionT1>
-          <distortionT2>0.0</distortionT2>
-        </plugin>
-      </sensor>
-    </gazebo>
-  </xacro:if>
-  <xacro:if value="${camera_simulation_type == 'stereo'}">
-    <!-- Gazebo plugin for Left Mono Camera -->
-    <gazebo reference="oak_left_camera_frame">
-      <sensor type="camera" name="oak_left_sensor">
-        <update_rate>${mono_update_rate}</update_rate>
-        <camera>
-          <horizontal_fov>1.2566370614359172</horizontal_fov> <!-- 72° HFOV in radians -->
-          <vertical_fov>0.8552113334772214</vertical_fov><!-- 49° VFOV in radians -->
-          <image>
-            <width>${mono_width}</width>
-            <height>${mono_height}</height>
-            <format>L8</format> <!-- Monochrome (grayscale) -->
-          </image>
-          <clip>
-            <near>0.196</near> <!-- Min focus 19.6cm -->
-            <far>100.0</far> <!-- Arbitrary max range -->
-          </clip>
-        </camera>
-        <plugin name="oak_left_camera_controller" filename="libgazebo_ros_camera.so">
-          <alwaysOn>true</alwaysOn>
-          <updateRate>${mono_update_rate}</updateRate>
-          <cameraName>oak_left</cameraName>
-          <frameName>oak_left_camera_optical_frame</frameName>
-          <imageTopicName>image_raw</imageTopicName>
-          <cameraInfoTopicName>camera_info</cameraInfoTopicName>
-          <distortionK1>0.0</distortionK1>
-          <distortionK2>0.0</distortionK2>
-          <distortionK3>0.0</distortionK3>
-          <distortionT1>0.0</distortionT1>
-          <distortionT2>0.0</distortionT2>
-        </plugin>
-      </sensor>
-    </gazebo>
-    <!-- Gazebo plugin for Right Mono Camera -->
-    <gazebo reference="oak_right_camera_frame">
-      <sensor type="camera" name="oak_right_sensor">
-        <update_rate>${mono_update_rate}</update_rate>
-        <camera>
-          <horizontal_fov>1.2566370614359172</horizontal_fov> <!-- 72° HFOV in radians -->
-          <vertical_fov>0.8552113334772214</vertical_fov><!-- 49° VFOV in radians -->
-          <image>
-            <width>${mono_width}</width>
-            <height>${mono_height}</height>
-            <format>L8</format> <!-- Monochrome (grayscale) -->
-          </image>
-          <clip>
-            <near>0.196</near> <!-- Min focus 19.6cm -->
-            <far>100.0</far> <!-- Arbitrary max range -->
-          </clip>
-        </camera>
-        <plugin name="oak_right_camera_controller" filename="libgazebo_ros_camera.so">
-          <alwaysOn>true</alwaysOn>
-          <updateRate>${mono_update_rate}</updateRate>
-          <cameraName>oak_right</cameraName>
-          <frameName>oak_right_camera_optical_frame</frameName>
-          <imageTopicName>image_raw</imageTopicName>
-          <cameraInfoTopicName>camera_info</cameraInfoTopicName>
-          <distortionK1>0.0</distortionK1>
-          <distortionK2>0.0</distortionK2>
-          <distortionK3>0.0</distortionK3>
-          <distortionT1>0.0</distortionT1>
-          <distortionT2>0.0</distortionT2>
-        </plugin>
-      </sensor>
-    </gazebo>
-  </xacro:if>
-  <xacro:if value="${camera_simulation_type == 'rgbd'}">
-    <!-- Depth Camera (Simulating RGB-D using stereo pair) -->
-    <link name="oak_depth_frame"/>
-    <joint name="oak_depth_joint" type="fixed">
-      <parent link="oak-d_frame"/>
-      <child link="oak_depth_frame"/>
-      <origin rpy="0 0 0" xyz="0 0 0"/> <!-- Centered on oak-d_frame -->
-    </joint>
-    <link name="oak_depth_optical_frame"/>
-    <joint name="oak_depth_optical_joint" type="fixed">
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