Commit message: Update mcm07_customization.urdf.xacro

File: catkin_ws/src/husky_oakd_stereo_nav/urdf/mcm07_customization.urdf.xacro (robot description, xacro)
@@ -43,5 +43,5 @@
     <parent link="base_link"/>
     <child link="D05"/>
-    <origin xyz="0.00 0.00 0.235" rpy="0 0 0"/>
+    <origin xyz="0.00 0.00 0.234" rpy="0 0 0"/>
   </joint>
 <!-- Ouster OS1-32 -->
